File: hardware/aprstracker/aprs.kicad_pcb (KiCad board)
At the start: 2 copper layers, 102 x 39.3 mm, 122 parts, among them IC1 ATMEGA8-AI, J1 SMA, J2 SMA, P1 CONN_6, P3 CONN_2, Q1 MMBT5551, Q2 MMBT5551, Q3 BCX54, Q4 BFR93A, Q5 BFR93A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

Commit message: [HW] Update pcb/sch/gps
Connections:
- U2 pad 10: N-0000039 (its old number) -> GND
Routing:
- net (no net): track 2.81 -> 0.27 mm, vias 1 -> 0
- net GND: vias 173 -> 174
